Commit message: fix bugs

File: src/rosbot_description/ros2_control/rosbot_system.ros2_control.xacro (robot description, xacro)
@@ -1,60 +1,75 @@
 <?xml version="1.0"?>
 <robot xmlns:xacro="http://www.ros.org/wiki/xacro">
-  <xacro:macro name="rosbot_system" params="name prefix use_fake_hardware:=^|false fake_sensor_commands:=^|false slowdown:=2.0">
+  <xacro:macro name="rosbot_system"
+    params="name serial_number:=^|000000000000
+    joint0_name:=^|joint0
+    joint1_name:=^|joint1
+    use_fake_hardware:=^|false
+    fake_sensor_commands:=^|false
+    slowdown:=2.0">
     <ros2_control name="${name}" type="system">
-      <hardware>
+        <hardware>
+            <xacro:if value="${use_fake_hardware}">
+              <plugin>fake_components/GenericSystem</plugin>
+              <param name="fake_sensor_commands">${fake_sensor_commands}</param>
+              <param name="state_following_offset">0.0</param>
+            </xacro:if>
+            <xacro:unless value="${use_fake_hardware}">
+              <plugin>odrive_hardware_interface/ODriveHardwareInterface</plugin>
+            </xacro:unless>
+        </hardware>
+        <joint name="${joint0_name}">
+            <command_interface name="velocity">
+              <param name="min">-1</param>
+              <param name="max">1</param>
+            </command_interface>
+            <command_interface name="position" />
+            <command_interface name="effort" />
+            <state_interface name="velocity"/>
+            <state_interface name="position"/>
+            <state_interface name="effort" />
+          <param name="serial_number">${serial_number}</param>
+          <param name="axis">0</param>
+          <param name="enable_watchdog">1</param>
+          <param name="watchdog_timeout">0.5</param>
+        </joint>
+        <joint name="${joint1_name}">
+            <command_interface name="velocity">
+              <param name="min">-1</param>
+              <param name="max">1</param>
+            </command_interface>
+            <command_interface name="position" />
+            <command_interface name="effort" />
+            <state_interface name="velocity"/>
+            <state_interface name="position"/>
+            <state_interface name="effort" />
+          <param name="serial_number">${serial_number}</param>
+          <param name="axis">1</param>
+          <param name="enable_watchdog">1</param>
+          <param name="watchdog_timeout">0.5</param>
+        </joint>
         <xacro:if value="${use_fake_hardware}">
-          <plugin>fake_components/GenericSystem</plugin>
-          <param name="fake_sensor_commands">${fake_sensor_commands}</param>
-          <param name="state_following_offset">0.0</param>
+             <sensor name="axis0">
+                <state_interface name="axis_error" />
+                <state_interface name="motor_error" />
+                <state_interface name="encoder_error" />
+                <state_interface name="controller_error" />
+                <state_interface name="fet_temperature" />
+                <state_interface name="motor_temperature" />
+             </sensor>
+             <sensor name="axis1">
+                <state_interface name="axis_error" />
+                <state_interface name="motor_error" />
+                <state_interface name="encoder_error" />
+                <state_interface name="controller_error" />
+                <state_interface name="fet_temperature" />
+                <state_interface name="motor_temperature" />
+             </sensor>
         </xacro:if>
-        <xacro:unless value="${use_fake_hardware}">
-          <plugin>odrive_hardware_interface/ODriveHardwareInterface</plugin>
-        </xacro:unless>
-      </hardware>
-      <joint name="left_wheel_joint">
-        <command_interface name="velocity">
-          <param name="min">-1</param>
-          <param name="max">1</param>
-        </command_interface>
-        <command_interface name="position" />
-        <command_interface name="effort" />
-        <state_interface name="velocity"/>
-        <state_interface name="position"/>
-        <state_interface name="effort" />
-        <param name="axis">0</param>
-        <param name="enable_watchdog">1</param>
-        <param name="watchdog_timeout">0.5</param>
-      </joint>
-      <sensor name="axis0">
-        <state_interface name="axis_error" />
-        <state_interface name="motor_error" />
-        <state_interface name="encoder_error" />
-        <state_interface name="controller_error" />
-        <state_interface name="fet_temperature" />
-        <state_interface name="motor_temperature" />
-      </sensor>
-      <joint name="right_wheel_joint">
-        <command_interface name="velocity">
-          <param name="min">-1</param>
-          <param name="max">1</param>
-        </command_interface>
-        <command_interface name="position" />
-        <command_interface name="effort" />
-        <state_interface name="velocity"/>
-        <state_interface name="position"/>
-        <state_interface name="effort" />
-        <param name="axis">1</param>
-        <param name="enable_watchdog">1</param>
-        <param name="watchdog_timeout">0.5</param>
-      </joint>
-      <sensor name="axis1">
-        <state_interface name="axis_error" />
-        <state_interface name="motor_error" />
-        <state_interface name="encoder_error" />
-        <state_interface name="controller_error" />
-        <state_interface name="fet_temperature" />
-        <state_interface name="motor_temperature" />
-      </sensor>
+         <xacro:unless value="${use_fake_hardware}">
+              <sensor name="odrv0">
+                <param name="serial_number">${serial_number}</param>
+            </sensor>
+         </xacro:unless>
     </ros2_control>
   </xacro:macro>

File: src/rosbot_description/urdf/rosbot.urdf.xacro (robot description, xacro)
@@ -4,5 +4,5 @@
   <!-- TODO is use_sim argument used in any way? -->
   <!-- <xacro:arg name="use_sim" default="false" /> -->
-  <xacro:arg name="use_fake_hardware" default="true" />
+  <xacro:arg name="use_fake_hardware" default="false" />
   <xacro:arg name="fake_sensor_commands" default="false" />
   <xacro:arg name="prefix" default="" />
@@ -10,7 +10,14 @@
   <xacro:include filename="$(find rosbot_description)/gazebo/rosbot.materials.xacro" />
   <xacro:include filename="$(find rosbot_description)/gazebo/rosbot.gazebo.xacro" />
-  <xacro:include filename="$(find rosbot_description)/ros2_control/rosbot_system.ros2_control.xacro" />
   <xacro:rosbot_links prefix="$(arg prefix)" />
   <xacro:rosbot_gazebo prefix="$(arg prefix)" />
+  <xacro:include filename="$(find rosbot_description)/ros2_control/rosbot_system.ros2_control.xacro" />
+  <xacro:rosbot_system
+    name="RosbotSystem"
+    joint0_name="$(arg prefix)left_wheel_joint"
+    joint1_name="$(arg prefix)right_wheel_joint"
+    use_fake_hardware="$(arg use_fake_hardware)"
+    fake_sensor_commands="$(arg fake_sensor_commands)" />
+<!--
   <xacro:rosbot_system
     name="RosbotSystem"
@@ -18,3 +25,9 @@
     use_fake_hardware="$(arg use_fake_hardware)"
     fake_sensor_commands="$(arg fake_sensor_commands)"/>
+  <xacro:include filename="$(find rosbot_description)/ros2_control/rosbot_system.ros2_control.xacro" />
+  <xacro:odrive_ros2_control
+    name="ODriveDiffBot"
+    joint0_name="$(arg prefix)left_wheel_joint"
+    joint1_name="$(arg prefix)right_wheel_joint" />
+-->
 </robot>
