Commit message: code redesign added flag for simulation

File: src/rosbot_description/gazebo/rosbot.gazebo.xacro (robot description, xacro)
@@ -96,11 +96,12 @@
     <!-- TODO use shared configuration, currently in rosbot_links.urdf.xacro -->
     <!-- http://gazebosim.org/tutorials?tut=ros_gzplugins -->
+    <!--
     <gazebo>
-      <plugin name='diff_drive' filename='libgazebo_ros_diff_drive.so'>
+      <plugin name='mini_base_diff_drive' filename='libgazebo_ros_diff_drive.so'>
         <update_rate>30</update_rate>
         <left_joint>left_wheel_joint</left_joint>
         <right_joint>right_wheel_joint</right_joint>
-        <wheel_separation>0.241</wheel_separation>
-        <wheel_diameter>0.195</wheel_diameter>
+        <wheel_separation>0.20</wheel_separation>
+        <wheel_diameter>0.170</wheel_diameter>
         <max_wheel_torque>50</max_wheel_torque>
         <max_wheel_acceleration>2.0</max_wheel_acceleration>
@@ -111,5 +112,12 @@
         <command_topic>cmd_vel</command_topic>
         <robot_base_frame>base_link</robot_base_frame>
-        <!-- <robot_base_frame>base_footprint</robot_base_frame> -->
+      </plugin>
+    </gazebo>
+    -->
+    <!-- ros_control plugin -->
+    <gazebo>
+      <plugin name="gazebo_ros2_control" filename="libgazebo_ros2_control.so">
+        <parameters>$(find rosbot_description)/config/robot_controllers.yaml</parameters>
+        <parameters>$(find rosbot_description)/config/robot_use_sim_param.yaml</parameters>
       </plugin>
     </gazebo>

File: src/rosbot_description/ros2_control/rosbot_system.ros2_control.xacro (robot description, xacro)
@@ -5,19 +5,33 @@
     joint0_name:=^|joint0
     joint1_name:=^|joint1
-    use_fake_hardware:=^|false
-    fake_sensor_commands:=^|false
+    use_gazebo:=^|true
     slowdown:=2.0">
     <ros2_control name="${name}" type="system">
+      <xacro:if value="$(arg use_gazebo)">
         <hardware>
-            <xacro:if value="${use_fake_hardware}">
-              <plugin>fake_components/GenericSystem</plugin>
-              <param name="fake_sensor_commands">${fake_sensor_commands}</param>
-              <param name="state_following_offset">0.0</param>
-            </xacro:if>
-            <xacro:unless value="${use_fake_hardware}">
+          <plugin>gazebo_ros2_control/GazeboSystem</plugin>
+        </hardware>
+      </xacro:if>
+      <xacro:unless value="$(arg use_gazebo)">
+        <hardware>
               <plugin>odrive_hardware_interface/ODriveHardwareInterface</plugin>
-            </xacro:unless>
         </hardware>
+      </xacro:unless>
         <joint name="${joint0_name}">
+            <command_interface name="velocity">
+              <param name="min">-1</param>
+              <param name="max">1</param>
+            </command_interface>
+            <command_interface name="position" />
+            <command_interface name="effort" />
+            <state_interface name="velocity"/>
+            <state_interface name="position"/>
+            <state_interface name="effort" />
+          <param name="serial_number">${serial_number}</param>
+          <param name="axis">1</param>
+          <param name="enable_watchdog">1</param>
+          <param name="watchdog_timeout">0.5</param>
+        </joint>
+        <joint name="${joint1_name}">
             <command_interface name="velocity">
               <param name="min">-1</param>
@@ -34,20 +48,6 @@
           <param name="watchdog_timeout">0.5</param>
         </joint>
-        <joint name="${joint1_name}">
-            <command_interface name="velocity">
-              <param name="min">-1</param>
-              <param name="max">1</param>
-            </command_interface>
-            <command_interface name="position" />
-            <command_interface name="effort" />
-            <state_interface name="velocity"/>
-            <state_interface name="position"/>
-            <state_interface name="effort" />
-          <param name="serial_number">${serial_number}</param>
-          <param name="axis">1</param>
-          <param name="enable_watchdog">1</param>
-          <param name="watchdog_timeout">0.5</param>
-        </joint>
-        <xacro:if value="${use_fake_hardware}">
+        <!-- -->
+        <xacro:if value="${use_gazebo}">
              <sensor name="axis0">
                 <state_interface name="axis_error" />
@@ -67,9 +67,10 @@
              </sensor>
         </xacro:if>
-         <xacro:unless value="${use_fake_hardware}">
+         <xacro:unless value="${use_gazebo}">
               <sensor name="odrv0">
                 <param name="serial_number">${serial_number}</param>
             </sensor>
          </xacro:unless>
+         <!-- -->
     </ros2_control>
   </xacro:macro>

File: src/rosbot_description/urdf/rosbot.urdf.xacro (robot description, xacro)
@@ -4,6 +4,5 @@
   <!-- TODO is use_sim argument used in any way? -->
   <!-- <xacro:arg name="use_sim" default="false" /> -->
-  <xacro:arg name="use_fake_hardware" default="false" />
-  <xacro:arg name="fake_sensor_commands" default="false" />
+  <xacro:arg name="use_gazebo" default="false" />
   <xacro:arg name="prefix" default="" />
   <xacro:include filename="$(find rosbot_description)/urdf/rosbot_links.urdf.xacro" />
@@ -17,17 +16,4 @@
     joint0_name="$(arg prefix)left_wheel_joint"
     joint1_name="$(arg prefix)right_wheel_joint"
-    use_fake_hardware="$(arg use_fake_hardware)"
-    fake_sensor_commands="$(arg fake_sensor_commands)" />
-<!--
-  <xacro:rosbot_system
-    name="RosbotSystem"
-    prefix="$(arg prefix)"
-    use_fake_hardware="$(arg use_fake_hardware)"
-    fake_sensor_commands="$(arg fake_sensor_commands)"/>
-  <xacro:include filename="$(find rosbot_description)/ros2_control/rosbot_system.ros2_control.xacro" />
-  <xacro:odrive_ros2_control
-    name="ODriveDiffBot"
-    joint0_name="$(arg prefix)left_wheel_joint"
-    joint1_name="$(arg prefix)right_wheel_joint" />
--->
+    use_gazebo="$(arg use_gazebo)" />
 </robot>

Commit message: update all changes

File: src/rosbot_description/gazebo/rosbot.gazebo.xacro (robot description, xacro)
@@ -126,5 +126,5 @@
       <sensor name="lidar" type="ray">
         <always_on>true</always_on>
-        <visualize>true</visualize>
+        <visualize>false</visualize>
         <update_rate>10</update_rate>
         <ray>

File: src/rosbot_description/urdf/rosbot_links.urdf.xacro (robot description, xacro)
@@ -16,5 +16,5 @@
     <xacro:property name="rear_wheel_mass" value="0.5" />
     <xacro:property name="rear_wheel_width" value="0.05" />
-    <xacro:property name="rear_wheel_radius" value="0.0975" />
+    <xacro:property name="rear_wheel_radius" value="0.085" />
     <xacro:property name="rear_wheel_origin_x" value="-0.1" />
     <xacro:property name="rear_wheel_distance" value="0.241" />
